File: hardware/suma-v-0-rev-a/suma-v-0-rev-a.kicad_sch (KiCad schematic)
At the start: 22 parts, among them J1 AudioJack2_SwitchT, J2 AudioJack2_SwitchT, J3 AudioJack2_SwitchT, J4 Conn_02x05_Odd_Even, J5 AudioJack2_SwitchT, J6 AudioJack2_SwitchT, U1 TL072

Commit message: agregar suma
Other:
- note added: ".tran 10u 40m"
