File: hardware/suma-v-0-rev-b/suma-v-0-rev-b.kicad_sch (KiCad schematic)
At the start: 22 parts, among them J1 AudioJack2_SwitchT, J2 AudioJack2_SwitchT, J3 AudioJack2_SwitchT, J4 Conn_02x05_Odd_Even, J5 AudioJack2_SwitchT, J6 AudioJack2_SwitchT, U1 TL072

Commit message: corregidos diodos y potes
Parts:
- removed J6: AudioJack2_SwitchT, suma-v-0-rev-b:Jack_3.5mm_QingPu_WQP-PJ398SM_Vertical, symbol suma-v-0-rev-b:AudioJack2_SwitchT
- removed R8: 1k, suma-v-0-rev-b:R0805, symbol suma-v-0-rev-b:R
- D1, D2: footprint suma-v-0-rev-b:SOD-123FL_L2.8-W1.8-LS3.7-R-RD -> popusintes:Diodo_SOD-123FL
- RV1, RV2, RV3: footprint suma-v-0-rev-b:POT_TH_Alps_RK09K_Single_Vertical -> popusintes:Potenciometro_Alpha_RD901F_Vertical
Connections:
- no-connect marks 2 -> 1
Other:
- note removed: "salida-invertida"
