File: hardware/suma-v-0-rev-b/suma-v-0-rev-b.kicad_pcb (KiCad board)
At the start: 2 copper layers, 25 x 100 mm, 22 parts, among them J1 AudioJack2_SwitchT, J2 AudioJack2_SwitchT, J3 AudioJack2_SwitchT, J4 Conn_02x05_Odd_Even, J5 AudioJack2_SwitchT, J6 AudioJack2_SwitchT, U1 TL072

Commit message: corregidos diodos y potes
Parts:
- removed J6: AudioJack2_SwitchT, suma-v-0-rev-b:Jack_3.5mm_QingPu_WQP-PJ398SM_Vertical
- removed R8: 1k, suma-v-0-rev-b:R0805
- D1, D2: footprint suma-v-0-rev-b:SOD-123FL_L2.8-W1.8-LS3.7-R-RD -> popusintes:Diodo_SOD-123FL
- RV1, RV2, RV3: footprint suma-v-0-rev-b:POT_TH_Alps_RK09K_Single_Vertical -> popusintes:Potenciometro_Alpha_RD901F_Vertical
Routing:
- net Net-(J5-Pad3): track 69.4 -> 0.00 mm
- net Net-(J6-Pad3): track 68.6 -> 0.00 mm
- net Net-(R3-Pad1): track 59.5 -> 0.00 mm, vias 2 -> 0
- net Net-(R2-Pad1): track 55.6 -> 0.00 mm, vias 3 -> 0
- net Net-(R4-Pad2): track 41.6 -> 0.00 mm, vias 4 -> 0
- net GND: track 40.7 -> 0.00 mm, vias 2 -> 0
- net Net-(U1A--): track 38.6 -> 0.00 mm, vias 3 -> 0
- net Net-(R1-Pad1): track 36.0 -> 0.00 mm, vias 1 -> 0
- net Net-(U1B--): track 24.4 -> 0.00 mm
- net Net-(J2-Pad3): track 20.8 -> 0.00 mm
- net Net-(J1-Pad3): track 20.8 -> 0.00 mm
- net Net-(J3-Pad3): track 20.5 -> 0.00 mm
- net Net-(R6-Pad2): track 19.7 -> 0.00 mm, vias 2 -> 0
- net -12V: track 17.6 -> 0.00 mm
- net Net-(D1-A): track 11.1 -> 0.00 mm
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
Commit message: agregar pcb
Parts:
- moved J4 0.70 mm to (37.6, 35.0)
Routing:
- net Net-(R3-Pad1): track 0.00 -> 62.0 mm
- net Net-(J5-Pad3): track 0.00 -> 58.3 mm
- net Net-(U1A--): track 0.00 -> 45.7 mm, vias 0 -> 3
- net Net-(R2-Pad1): track 0.00 -> 44.5 mm, vias 0 -> 1
- net Net-(R1-Pad1): track 0.00 -> 29.7 mm, vias 0 -> 1
- net Net-(R4-Pad2): track 0.00 -> 24.6 mm, vias 0 -> 3
- net -12V: track 0.00 -> 21.7 mm
- net Net-(R6-Pad2): track 0.00 -> 19.3 mm
- net Net-(J2-Pad3): track 0.00 -> 16.1 mm
- net Net-(J3-Pad3): track 0.00 -> 16.1 mm
- net Net-(U1B--): track 0.00 -> 16.0 mm
- net Net-(J1-Pad3): track 0.00 -> 15.9 mm
- net +12V: track 0.00 -> 10.9 mm
- net Net-(D1-A): track 0.00 -> 10.2 mm
- net Net-(D2-K): track 0.00 -> 9.78 mm
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
Commit message: rev-b docs
Parts:
- moved C2 3.98 mm to (36.0, 47.0)
Routing:
- net GND: track 5.83 -> 30.2 mm, vias 2 -> 4
- net -12V: track 21.7 -> 17.2 mm
Changed lines of the file:
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@@
 	(footprint "suma-v-0-rev-b:C0805"
 		(layer "F.Cu")
-		(at 33.5 43.9)
+		(at 36 47)
 		(descr "1uF (105) ±10% 50V")
 		(property "Reference" "C2"
-			(at -0.1 -1.8 0)
+			(at -2 -1.8 0)
 			(layer "F.SilkS")
 			(effects
@@
 		)
 	)
-	(segment
-		(start 47 59)
-		(end 46 59)
-		(width 0.2)
-		(layer "F.Cu")
+	(via
+		(at 41 82)
+		(size 0.6)
+		(drill 0.3)
+		(layers "F.Cu" "B.Cu")
 		(net "GND")
 	)
@@
 		(net "GND")
 	)
+	(via
+		(at 40 99)
+		(size 0.6)
+		(drill 0.3)
+		(layers "F.Cu" "B.Cu")
+		(net "GND")
+	)
 	(segment
 		(start 46 59)
@@
 	)
 	(segment
+		(start 53 98)
+		(end 41 98)
+		(width 0.2)
+		(layer "B.Cu")
+		(net "GND")
+	)
+	(segment
+		(start 41 98)
+		(end 40 99)
+		(width 0.2)
+		(layer "B.Cu")
+		(net "GND")
+	)
+	(segment
+		(start 53 82)
+		(end 41 82)
+		(width 0.2)
+		(layer "B.Cu")
+		(net "GND")
+	)
+	(segment
 		(start 45 62)
 		(end 46 63)
@@
 	)
 	(segment
-		(start 40 47)
-		(end 37.6 47)
+		(start 38 55.312)
+		(end 39.188 56.5)
 		(width 0.8)
 		(layer "F.Cu")
@@
 	)
 	(segment
-		(start 40.59 46.41)
-		(end 40 47)
+		(start 37 47)
+		(end 37 51)
 		(width 0.8)
 		(layer "F.Cu")
@@
 	)
 	(segment
-		(start 38.5 56.5)
-		(end 38 56)
+		(start 40.59 45.41)
+		(end 40.59 44)
 		(width 0.8)
 		(layer "F.Cu")
@@
 	)
 	(segment
-		(start 37.6 47)
-		(end 34.5 43.9)
+		(start 39.188 56.5)
+		(end 40.3 56.5)
 		(width 0.8)
 		(layer "F.Cu")
@@
 	)
 	(segment
-		(start 38 56)
-		(end 38 47.4)
+		(start 37 47)
+		(end 39 47)
 		(width 0.8)
 		(layer "F.Cu")
@@
 	)
 	(segment
-		(start 40.3 56.5)
-		(end 38.5 56.5)
+		(start 37 51)
+		(end 38 52)
 		(width 0.8)
 		(layer "F.Cu")
@@
 	)
 	(segment
-		(start 38 47.4)
-		(end 37.6 47)
+		(start 38 52)
+		(end 38 55.312)
 		(width 0.8)
 		(layer "F.Cu")
@@
 	)
 	(segment
-		(start 40.59 44)
-		(end 40.59 46.41)
+		(start 39 47)
+		(end 40.59 45.41)
 		(width 0.8)
 		(layer "F.Cu")
